Commit message: Add g1 variants

File: urdf/g1_29dof.urdf (robot description, URDF)
Before this commit: robot g1_29dof, 40 links, 39 joints
Links:
- link left_rubber_hand: geometry collision mesh filename=package://g1_description/meshes/left_rubber_hand.STL; visual mesh filename=package://g1_description/meshes/left_rubber_hand.STL
- link right_rubber_hand: geometry collision mesh filename=package://g1_description/meshes/right_rubber_hand.STL; visual mesh filename=package://g1_description/meshes/right_rubber_hand.STL
